Commit message: Change ucar_bringup ucar_navigation

File: src/urdf_rviz/urdf/xacro/car.urdf.xacro (robot description, xacro)
@@ -4,5 +4,5 @@
     <xacro:include filename="$(find velodyne_description)/urdf/VLP-16.urdf.xacro" />
     <!-- 引用imu的xacro文件 -->
-    <xacro:include filename="$(find urdf01_rviz)/urdf/xacro/imu_gazebo.xacro" />
+    <xacro:include filename="$(find urdf_rviz)/urdf/xacro/imu_gazebo.xacro" />
     <!-- 封装变量、常量 -->
     <xacro:property name="PI" value="3.14159265358979"/>
@@ -46,5 +46,5 @@
     <!-- 添加 IMU 模型 -->
     <xacro:property name="imu_hight" value="0.05" />
-    <xacro:property name="imu_x" value="0.0" />
+    <xacro:property name="imu_x" value="-0.08" />
     <xacro:property name="imu_y" value="0.0" />
     <xacro:property name="imu_z" value="${base_link_length / 2 + imu_hight / 2}" />
@@ -55,4 +55,11 @@
         <child link="imu_link" />
         <origin xyz="${imu_x} ${imu_y} ${imu_z}" rpy="0 0 0" />
+        <visual>
+            <origin rpy="0 0 0" xyz="${imu_x} ${imu_y} ${imu_z}" />
+            <geometry>
+                <box size="${imu_size} ${imu_size} ${imu_size}"/>
+            </geometry>
+            <material name="red"/>
+        </visual>
     </joint>
     <!-- 驱动轮属性 -->
@@ -136,5 +143,3 @@
         <origin xyz="${laser_x} ${laser_y} ${laser_z}" />
     </joint>
-    <!-- 调用 VLP-16 雷达宏 -->
-    <xacro:VLP-16 parent="velodyne_base_link" name="velodyne" topic="/velodyne_points" organize_cloud="false" hz="10" lasers="16" samples="1875" collision_range="0.3" min_range="0.9" max_range="130.0" noise="0.008" min_angle="-${PI}" max_angle="${PI}" gpu="true" />
 </robot>

File: src/urdf_rviz/urdf/xacro/imu_gazebo.xacro (robot description, xacro)
@@ -30,5 +30,5 @@
             <sensor name="imu_sensor" type="imu">
                 <always_on>true</always_on>
-                <update_rate>500</update_rate>
+                <update_rate>100</update_rate>
                 <visualize>true</visualize>
                 <topic>__default_topic__</topic>
@@ -36,5 +36,5 @@
                     <topicName>imu</topicName>
                     <bodyName>imu_link</bodyName>
-                    <updateRateHZ>500.0</updateRateHZ>
+                    <updateRateHZ>100.0</updateRateHZ>
                     <gaussianNoise>0.0</gaussianNoise>
                     <xyzOffset>0 0 0</xyzOffset>
