Commit message: 更新imu_gazebo以添加父链接；添加laser_support并以调用形式在robot_car中对velodyne-16进行调用，而不是使用仿真文件

File: src/robot_description/urdf/imu_gazebo.xacro (robot description, xacro)
@@ -7,4 +7,5 @@
     <xacro:property name="imu_y"        value="0.0" />
     <xacro:property name="imu_z"        value="0.0" />
+    <!-- 默认惯性参数 -->
     <xacro:macro name="default_inertial" params="mass">
         <inertial>
@@ -13,5 +14,7 @@
         </inertial>
     </xacro:macro>
+    <!-- IMU 传感器宏 -->
     <xacro:macro name="imu" params="prefix:=imu">
+        <!-- IMU 链接 -->
         <link name="imu_link">
             <visual>
@@ -26,4 +29,11 @@
             </collision>
         </link>
+        <!-- 关节连接 imu_link 和 base_link -->
+        <joint name="imu_to_base" type="fixed">
+            <parent link="base_link"/>
+            <child link="imu_link"/>
+            <origin rpy="0 0 0" xyz="${imu_x} ${imu_y} ${imu_z}"/>
+        </joint>
+        <!-- Gazebo 配置 -->
         <gazebo reference="${prefix}_link">
             <gravity>true</gravity>

File: src/robot_description/urdf/robot_car.xacro (robot description, xacro)
@@ -4,8 +4,16 @@
     <xacro:include filename="my_base.urdf.xacro" />
     <xacro:include filename="my_camera.urdf.xacro" />
-    <xacro:include filename="my_laser.urdf.xacro" />
+    <!-- 更新结构信息，以laser_support + velodyne 为构建，不需要自己写雷达仿真的xacro文件 -->
+    <!-- <xacro:include filename="my_laser.urdf.xacro" /> -->
     <xacro:include filename="move.urdf.xacro" />
+    <xacro:include filename="imu_gazebo.xacro" />
     <!-- 雷达仿真的 xacro 文件 -->
-    <xacro:include filename="my_sensors_laser.urdf.xacro" />
+    <!-- <xacro:include filename="my_sensors_laser.urdf.xacro" /> -->
+    <!-- VLP16 激光雷达 -->
+    <xacro:include filename="$(find robot_description)/urdf/laser_support.xacro" />
+    <xacro:include filename="$(find velodyne_description)/urdf/VLP-16.urdf.xacro"/>
+    <xacro:VLP-16 parent="support" name="velodyne" topic="/velodyne_points" organize_cloud="${organize_cloud}" hz="10" samples="440" gpu="${gpu}">
+          <origin xyz="0 0 ${support_length/2}" rpy="0 0 0" />
+    </xacro:VLP-16>
     <!-- 摄像头仿真的 xacro 文件 -->
     <xacro:include filename="my_sensors_camara.urdf.xacro" />
