Commit message: 整合摄像头模块和IMU模块，更改IMU模块名字

File: src/robot_description/urdf/my_camera.xacro (robot description, xacro)
@@ -1,11 +1,11 @@
-<!-- 摄像头相关的 xacro 文件 -->
-<robot name="my_camera" xmlns:xacro="http://wiki.ros.org/xacro">
+<?xml version="1.0"?>
+<robot name="my_camera" xmlns:xacro="http://www.ros.org/wiki/xacro">
     <!-- 摄像头属性 -->
-    <xacro:property name="camera_length" value="0.01" /> <!-- 摄像头长度(x) -->
-    <xacro:property name="camera_width" value="0.025" /> <!-- 摄像头宽度(y) -->
-    <xacro:property name="camera_height" value="0.025" /> <!-- 摄像头高度(z) -->
-    <xacro:property name="camera_x" value="0.08" /> <!-- 摄像头安装的x坐标 -->
-    <xacro:property name="camera_y" value="0.0" /> <!-- 摄像头安装的y坐标 -->
-    <xacro:property name="camera_z" value="${base_link_length / 2 + camera_height / 2}" /> <!-- 摄像头安装的z坐标:底盘高度 / 2 + 摄像头高度 / 2  -->
+    <xacro:property name="camera_length"    value="0.01" /> <!-- 摄像头长度(x) -->
+    <xacro:property name="camera_width"     value="0.025" /> <!-- 摄像头宽度(y) -->
+    <xacro:property name="camera_height"    value="0.025" /> <!-- 摄像头高度(z) -->
+    <xacro:property name="camera_x"         value="0.08" /> <!-- 摄像头安装的x坐标 -->
+    <xacro:property name="camera_y"         value="0.0" /> <!-- 摄像头安装的y坐标 -->
+    <xacro:property name="camera_z"         value="${base_link_length / 2 + camera_height / 2}" /> <!-- 摄像头安装的z坐标:底盘高度 / 2 + 摄像头高度 / 2  -->
     <xacro:property name="camera_m" value="0.01" /> <!-- 摄像头质量 -->
     <!-- 摄像头关节以及link -->
@@ -31,6 +31,42 @@
         <origin xyz="${camera_x} ${camera_y} ${camera_z}" />
     </joint>
+    <!-- Gazebo 配置 -->
     <gazebo reference="camera">
-        <material>Gazebo/Blue</material>
+        <!-- 摄像头传感器 -->
+        <sensor type="camera" name="camera_node">
+            <update_rate>30.0</update_rate> <!-- 更新频率 -->
+            <camera name="head">
+                <horizontal_fov>1.3962634</horizontal_fov> <!-- 水平视场角 (80°) -->
+                <image>
+                    <width>1280</width>
+                    <height>720</height>
+                    <format>R8G8B8</format>
+                </image>
+                <clip>
+                    <near>0.02</near>
+                    <far>300</far>
+                </clip>
+                <noise>
+                    <type>gaussian</type>
+                    <mean>0.0</mean>
+                    <stddev>0.007</stddev>
+                </noise>
+            </camera>
+            <!-- 核心插件 -->
+            <plugin name="gazebo_camera" filename="libgazebo_ros_camera.so">
+                <alwaysOn>true</alwaysOn>
+                <updateRate>0.0</updateRate>
+                <cameraName>/camera</cameraName>
+                <imageTopicName>image_raw</imageTopicName>
+                <cameraInfoTopicName>camera_info</cameraInfoTopicName>
+                <frameName>camera</frameName>
+                <hackBaseline>0.07</hackBaseline>
+                <distortionK1>0.0</distortionK1>
+                <distortionK2>0.0</distortionK2>
+                <distortionK3>0.0</distortionK3>
+                <distortionT1>0.0</distortionT1>
+                <distortionT2>0.0</distortionT2>
+            </plugin>
+        </sensor>
     </gazebo>
 </robot>

File: src/robot_description/urdf/my_imu.xacro (robot description, xacro)
@@ -2,9 +2,10 @@
 <robot xmlns:xacro="http://www.ros.org/wiki/xacro" name="imu">
     <!-- IMU 属性 -->
-    <xacro:property name="imu_size"     value="0.1" />
-    <xacro:property name="imu_hight"    value="0.1" />
-    <xacro:property name="imu_x"        value="0.0" />
+    <xacro:property name="imu_length"   value="0.02" /> <!-- IMU长度(x) -->
+    <xacro:property name="imu_width"    value="0.025" /> <!-- IMU宽度(y) -->
+    <xacro:property name="imu_height"   value="0.03" /> <!-- IMU高度(z) -->
+    <xacro:property name="imu_x"        value="-0.08" />
     <xacro:property name="imu_y"        value="0.0" />
-    <xacro:property name="imu_z"        value="0.0" />
+    <xacro:property name="imu_z"        value="${base_link_length / 2 + imu_height / 2}" />
     <!-- 默认惯性参数 -->
     <xacro:macro name="default_inertial" params="mass">
@@ -21,10 +22,10 @@
                <origin rpy="0 0 0" xyz="${imu_x} ${imu_y} ${imu_z}" />
                <geometry>
-                    <box size="${imu_size} ${imu_size} ${imu_size}"/>
+                    <box size="${imu_length} ${imu_width} ${imu_height}"/>
                </geometry>
               <material name="red"/>
             </visual>
             <collision>
-                <box size="${imu_size} ${imu_size} ${imu_size}"/>
+                <box size="${imu_length} ${imu_length} ${imu_height}"/>
             </collision>
         </link>

File: src/robot_description/urdf/robot_car.xacro (robot description, xacro)
@@ -1,11 +1,10 @@
 <!-- 组合小车底盘与传感器 -->
 <robot name="my_car_camera" xmlns:xacro="http://wiki.ros.org/xacro">
-    <xacro:include filename="my_head.urdf.xacro" />
-    <xacro:include filename="my_base.urdf.xacro" />
-    <xacro:include filename="my_camera.urdf.xacro" />
+    <xacro:include filename="$(find robot_description)/urdf/my_head.urdf.xacro" />
+    <xacro:include filename="$(find robot_description)/urdf/my_base.urdf.xacro" />
+    <xacro:include filename="$(find robot_description)/urdf/my_camera.urdf.xacro" />
+    <xacro:include filename="$(find robot_description)/urdf/move.urdf.xacro" />
     <!-- 更新结构信息，以laser_support + velodyne 为构建，不需要自己写雷达仿真的xacro文件 -->
     <!-- <xacro:include filename="my_laser.urdf.xacro" /> -->
-    <xacro:include filename="move.urdf.xacro" />
-    <xacro:include filename="imu_gazebo.xacro" />
     <!-- 雷达仿真的 xacro 文件 -->
     <!-- <xacro:include filename="my_sensors_laser.urdf.xacro" /> -->
@@ -16,5 +15,7 @@
           <origin xyz="0 0 ${support_length/2}" rpy="0 0 0" />
     </xacro:VLP-16>
-    <!-- 摄像头仿真的 xacro 文件 -->
-    <xacro:include filename="my_sensors_camara.urdf.xacro" />
+    <!-- IMU 模块 -->
+    <xacro:include filename="$(find robot_description)/urdf/my_imu.xacro"/>
+    <!-- 摄像头模块 -->
+    <xacro:include filename="$(find robot_description)/urdf/my_camera.xacro" />
 </robot>
