Commit message: Depart discribe of car.xacro

File: src/robot_description/urdf/move.xacro (robot description, xacro)
@@ -1,4 +1,6 @@
-<robot name="move" xmlns:xacro="http://wiki.ros.org/xacro">
+<robot name="my_car_move" xmlns:xacro="http://wiki.ros.org/xacro">
+    <!-- 传动实现:用于连接控制器与关节 -->
     <xacro:macro name="joint_trans" params="joint_name">
+        <!-- Transmission is important to link the joints and the controller -->
         <transmission name="${joint_name}_trans">
             <type>transmission_interface/SimpleTransmission</type>
@@ -12,6 +14,8 @@
         </transmission>
     </xacro:macro>
+    <!-- 每一个驱动轮都需要配置传动装置 -->
     <xacro:joint_trans joint_name="left_wheel2base_link" />
     <xacro:joint_trans joint_name="right_wheel2base_link" />
+    <!-- 控制器 -->
     <gazebo>
         <plugin name="differential_drive_controller" filename="libgazebo_ros_diff_drive.so">
@@ -24,15 +28,15 @@
             <updateRate>100.0</updateRate>
             <legacyMode>true</legacyMode>
-            <leftJoint>left_wheel2base_link</leftJoint>
-            <rightJoint>right_wheel2base_link</rightJoint>
-            <wheelSeparation>${base_link_radius * 2}</wheelSeparation>
-            <wheelDiameter>${wheel_radius * 2}</wheelDiameter>
+            <leftJoint>left_wheel2base_link</leftJoint> <!-- 左轮 -->
+            <rightJoint>right_wheel2base_link</rightJoint> <!-- 右轮 -->
+            <wheelSeparation>${base_link_radius * 2}</wheelSeparation> <!-- 车轮间距 -->
+            <wheelDiameter>${wheel_radius * 2}</wheelDiameter> <!-- 车轮直径 -->
             <broadcastTF>1</broadcastTF>
             <wheelTorque>30</wheelTorque>
             <wheelAcceleration>1.8</wheelAcceleration>
-            <commandTopic>cmd_vel</commandTopic>
+            <commandTopic>cmd_vel</commandTopic> <!-- 运动控制话题 -->
             <odometryFrame>odom</odometryFrame>
-            <odometryTopic>odom</odometryTopic>
-            <robotBaseFrame>base_footprint</robotBaseFrame>
+            <odometryTopic>odom</odometryTopic> <!-- 里程计话题 -->
+            <robotBaseFrame>base_footprint</robotBaseFrame> <!-- 根坐标系 -->
         </plugin>
     </gazebo>

File: src/robot_description/urdf/my_base.xacro (robot description, xacro)
@@ -1,12 +1,25 @@
-<robot name="robot_base" xmlns:xacro="http://www.ros.org/wiki/xacro">
+<!--
+    使用 xacro 优化 URDF 版的小车底盘实现：
+    实现思路:
+    1.将一些常量、变量封装为 xacro:property
+      比如:PI 值、小车底盘半径、离地间距、车轮半径、宽度 ....
+    2.使用 宏 封装驱动轮以及支撑轮实现，调用相关宏生成驱动轮与支撑轮
+-->
+<!-- 根标签，必须声明 xmlns:xacro -->
+<robot name="my_base" xmlns:xacro="http://www.ros.org/wiki/xacro">
+    <!-- 封装变量、常量 -->
+    <!-- PI 值设置精度需要高一些，否则后续车轮翻转量计算时，可能会出现肉眼不能察觉的车轮倾斜，从而导致模型抖动 -->
     <xacro:property name="PI" value="3.1415926"/>
+    <!-- 宏:黑色设置 -->
     <material name="black">
         <color rgba="0.0 0.0 0.0 1.0" />
     </material>
-    <xacro:property name="base_footprint_radius" value="0.001" />
-    <xacro:property name="base_link_radius" value="0.1" />
-    <xacro:property name="base_link_length" value="0.08" />
-    <xacro:property name="earth_space" value="0.015" />
-    <xacro:property name="base_link_m" value="0.5" />
+    <!-- 底盘属性 -->
+    <xacro:property name="base_footprint_radius" value="0.001" /> <!-- base_footprint 半径  -->
+    <xacro:property name="base_link_radius" value="0.1" /> <!-- base_link 半径 -->
+    <xacro:property name="base_link_length" value="0.08" /> <!-- base_link 长 -->
+    <xacro:property name="earth_space" value="0.015" /> <!-- 离地间距 -->
+    <xacro:property name="base_link_m" value="0.5" /> <!-- 质量  -->
+    <!-- 底盘 -->
     <link name="base_footprint">
       <visual>
@@ -42,7 +55,10 @@
         <material>Gazebo/Yellow</material>
     </gazebo>
-    <xacro:property name="wheel_radius" value="0.0325" />
-    <xacro:property name="wheel_length" value="0.015" />
-    <xacro:property name="wheel_m" value="0.05" />
+    <!-- 驱动轮 -->
+    <!-- 驱动轮属性 -->
+    <xacro:property name="wheel_radius" value="0.0325" /><!-- 半径 -->
+    <xacro:property name="wheel_length" value="0.015" /><!-- 宽度 -->
+    <xacro:property name="wheel_m" value="0.05" /> <!-- 质量  -->
+    <!-- 驱动轮宏实现 -->
     <xacro:macro name="add_wheels" params="name flag">
       <link name="${name}_wheel">
@@ -74,6 +90,9 @@
     <xacro:add_wheels name="left" flag="1" />
     <xacro:add_wheels name="right" flag="-1" />
-    <xacro:property name="support_wheel_radius" value="0.0075" />
-    <xacro:property name="support_wheel_m" value="0.03" />
+    <!-- 支撑轮 -->
+    <!-- 支撑轮属性 -->
+    <xacro:property name="support_wheel_radius" value="0.0075" /> <!-- 支撑轮半径 -->
+    <xacro:property name="support_wheel_m" value="0.03" /> <!-- 质量  -->
+    <!-- 支撑轮宏 -->
     <xacro:macro name="add_support_wheel" params="name flag" >
       <link name="${name}_wheel">

File: src/robot_description/urdf/my_camera.xacro (robot description, xacro)
@@ -1,10 +1,13 @@
-<robot name="camera" xmlns:xacro="http://wiki.ros.org/xacro">
-    <xacro:property name="camera_length" value="0.01" />
-    <xacro:property name="camera_width" value="0.025" />
-    <xacro:property name="camera_height" value="0.025" />
-    <xacro:property name="camera_x" value="0.08" />
-    <xacro:property name="camera_y" value="0.0" />
-    <xacro:property name="camera_z" value="${base_link_length / 2 + camera_height / 2}" />
-    <xacro:property name="camera_m" value="0.01" />
+<!-- 摄像头相关的 xacro 文件 -->
+<robot name="my_camera" xmlns:xacro="http://wiki.ros.org/xacro">
+    <!-- 摄像头属性 -->
+    <xacro:property name="camera_length" value="0.01" /> <!-- 摄像头长度(x) -->
+    <xacro:property name="camera_width" value="0.025" /> <!-- 摄像头宽度(y) -->
+    <xacro:property name="camera_height" value="0.025" /> <!-- 摄像头高度(z) -->
+    <xacro:property name="camera_x" value="0.08" /> <!-- 摄像头安装的x坐标 -->
+    <xacro:property name="camera_y" value="0.0" /> <!-- 摄像头安装的y坐标 -->
+    <xacro:property name="camera_z" value="${base_link_length / 2 + camera_height / 2}" /> <!-- 摄像头安装的z坐标:底盘高度 / 2 + 摄像头高度 / 2  -->
+    <xacro:property name="camera_m" value="0.01" /> <!-- 摄像头质量 -->
+    <!-- 摄像头关节以及link -->
     <link name="camera">
         <visual>

File: src/robot_description/urdf/my_head.xacro (robot description, xacro)
@@ -1,2 +1,3 @@
+<?xml version="1.0"?>
 <robot name="inertia" xmlns:xacro="http://wiki.ros.org/xacro">
     <!-- Macro for inertia matrix -->

File: src/robot_description/urdf/my_laser.xacro (robot description, xacro)
@@ -1,9 +1,13 @@
-<robot name="laser" xmlns:xacro="http://wiki.ros.org/xacro">
-    <xacro:property name="support_length" value="0.15" />
-    <xacro:property name="support_radius" value="0.01" />
-    <xacro:property name="support_x" value="0.0" />
-    <xacro:property name="support_y" value="0.0" />
-    <xacro:property name="support_z" value="${base_link_length / 2 + support_length / 2}" />
-    <xacro:property name="support_m" value="0.02" />
+<!--
+    小车底盘添加雷达
+-->
+<robot name="my_laser" xmlns:xacro="http://wiki.ros.org/xacro">
+    <!-- 雷达支架 -->
+    <xacro:property name="support_length" value="0.15" /> <!-- 支架长度 -->
+    <xacro:property name="support_radius" value="0.01" /> <!-- 支架半径 -->
+    <xacro:property name="support_x" value="0.0" /> <!-- 支架安装的x坐标 -->
+    <xacro:property name="support_y" value="0.0" /> <!-- 支架安装的y坐标 -->
+    <xacro:property name="support_z" value="${base_link_length / 2 + support_length / 2}" /> <!-- 支架安装的z坐标:底盘高度 / 2 + 支架高度 / 2  -->
+    <xacro:property name="support_m" value="0.02" /> <!-- 支架质量 -->
     <link name="support">
         <visual>
@@ -32,10 +36,12 @@
         <material>Gazebo/White</material>
     </gazebo>
-    <xacro:property name="laser_length" value="0.05" />
-    <xacro:property name="laser_radius" value="0.03" />
-    <xacro:property name="laser_x" value="0.0" />
-    <xacro:property name="laser_y" value="0.0" />
-    <xacro:property name="laser_z" value="${support_length / 2 + laser_length / 2}" />
-    <xacro:property name="laser_m" value="0.1" />
+    <!-- 雷达属性 -->
+    <xacro:property name="laser_length" value="0.05" /> <!-- 雷达长度 -->
+    <xacro:property name="laser_radius" value="0.03" /> <!-- 雷达半径 -->
+    <xacro:property name="laser_x" value="0.0" /> <!-- 雷达安装的x坐标 -->
+    <xacro:property name="laser_y" value="0.0" /> <!-- 雷达安装的y坐标 -->
+    <xacro:property name="laser_z" value="${support_length / 2 + laser_length / 2}" /> <!-- 雷达安装的z坐标:支架高度 / 2 + 雷达高度 / 2  -->
+    <xacro:property name="laser_m" value="0.1" /> <!-- 雷达质量 -->
+    <!-- 雷达关节以及link -->
     <link name="laser">
         <visual>
@@ -62,19 +68,3 @@
         <material>Gazebo/Black</material>
     </gazebo>
-    <!-- 激光雷达插件 -->
-    <gazebo reference="laser">
-        <plugin name="gazebo_laser_plugin" filename="libgazebo_ros_laser.so">
-            <!-- 激光雷达的 ROS 话题名称 -->
-            <rosparam name="topic_name">scan</rosparam>
-            <!-- 激光雷达发布的传感器类型 -->
-            <rosparam name="frame_name">laser_frame</rosparam>
-            <!-- 激光雷达的最大范围和最小范围 -->
-            <rosparam name="laser_scan_range_max">10.0</rosparam>
-            <rosparam name="laser_scan_range_min">0.1</rosparam>
-            <!-- 激光雷达扫描的角度范围 -->
-            <rosparam name="horizontal_fov">1.57</rosparam> <!-- 90 degrees -->
-            <!-- 激光雷达的扫描频率 -->
-            <rosparam name="update_rate">10.0</rosparam>
-        </plugin>
-    </gazebo>
 </robot>

File: src/robot_description/urdf/robot_car.xacro (robot description, xacro)
@@ -1,7 +1,12 @@
-<robot name="robot_car" xmlns:xacro="http://wiki.ros.org/xacro">
-    <xacro:include filename="inertia.xacro" />
-    <xacro:include filename="robot_base.xacro" />
-    <xacro:include filename="camera.xacro" />
-    <xacro:include filename="laser.xacro" />
-    <xacro:include filename="move.xacro" />
+<!-- 组合小车底盘与传感器 -->
+<robot name="my_car_camera" xmlns:xacro="http://wiki.ros.org/xacro">
+    <xacro:include filename="my_head.urdf.xacro" />
+    <xacro:include filename="my_base.urdf.xacro" />
+    <xacro:include filename="my_camera.urdf.xacro" />
+    <xacro:include filename="my_laser.urdf.xacro" />
+    <xacro:include filename="move.urdf.xacro" />
+    <!-- 雷达仿真的 xacro 文件 -->
+    <xacro:include filename="my_sensors_laser.urdf.xacro" />
+    <!-- 摄像头仿真的 xacro 文件 -->
+    <xacro:include filename="my_sensors_camara.urdf.xacro" />
 </robot>

Commit message: 成功完成多传感器模型创建

File: src/robot_description/urdf/move.xacro (robot description, xacro)
@@ -21,8 +21,8 @@
         <plugin name="differential_drive_controller" filename="libgazebo_ros_diff_drive.so">
             <rosDebugLevel>Debug</rosDebugLevel>
-            <publishWheelTF>true</publishWheelTF>
+            <publishWheelTF>false</publishWheelTF> <!-- true 改 false 避免冲突 -->
             <robotNamespace>/</robotNamespace>
             <publishTf>1</publishTf>
-            <publishWheelJointState>true</publishWheelJointState>
+            <publishWheelJointState>false</publishWheelJointState> <!-- true 改 false 避免冲突 -->
             <alwaysOn>true</alwaysOn>
             <updateRate>100.0</updateRate>

File: src/robot_description/urdf/my_imu.xacro (robot description, xacro)
@@ -2,10 +2,11 @@
 <robot xmlns:xacro="http://www.ros.org/wiki/xacro" name="imu">
     <!-- IMU 属性 -->
-    <xacro:property name="imu_length"   value="0.02" /> <!-- IMU长度(x) -->
+    <xacro:property name="imu_length"   value="0.01" /> <!-- IMU长度(x) -->
     <xacro:property name="imu_width"    value="0.025" /> <!-- IMU宽度(y) -->
-    <xacro:property name="imu_height"   value="0.03" /> <!-- IMU高度(z) -->
+    <xacro:property name="imu_height"   value="0.025" /> <!-- IMU高度(z) -->
     <xacro:property name="imu_x"        value="-0.08" />
     <xacro:property name="imu_y"        value="0.0" />
     <xacro:property name="imu_z"        value="${base_link_length / 2 + imu_height / 2}" />
+    <xacro:property name="imu_m" value="0.01" /> <!-- IMU质量 -->
     <!-- 默认惯性参数 -->
     <xacro:macro name="default_inertial" params="mass">
@@ -20,13 +21,17 @@
         <link name="imu_link">
             <visual>
-               <origin rpy="0 0 0" xyz="${imu_x} ${imu_y} ${imu_z}" />
-               <geometry>
+                <geometry>
                     <box size="${imu_length} ${imu_width} ${imu_height}"/>
-               </geometry>
-              <material name="red"/>
+                </geometry>
+                <origin rpy="0 0 0" xyz="0 0 0" />
+                <material name="red"/>
             </visual>
             <collision>
-                <box size="${imu_length} ${imu_length} ${imu_height}"/>
+                <geometry>
+                    <box size="${imu_length} ${imu_width} ${imu_height}"/>
+                </geometry>
+                <origin rpy="0 0 0" xyz="0 0 0" />
             </collision>
+            <xacro:Box_inertial_matrix m="${imu_m}" l="${imu_length}" w="${imu_width}" h="${imu_height}" />
         </link>
         <!-- 关节连接 imu_link 和 base_link -->

File: src/robot_description/urdf/robot_car.urdf (robot description, URDF)
Before this commit: robot my_car_camera, 10 links, 9 joints
Links:
- added link imu_link; visual box size=0.01 0.025 0.0325
Joints:
- added joint imu_to_base: type fixed, parent base_link, child imu_link, origin xyz=-0.08 0.0 0.05625 rpy=0 0 0

File: src/robot_description/urdf/robot_car.xacro (robot description, xacro)
@@ -1,12 +1,13 @@
 <!-- 组合小车底盘与传感器 -->
-<robot name="my_car_camera" xmlns:xacro="http://wiki.ros.org/xacro">
+<robot name="robot_car" xmlns:xacro="http://wiki.ros.org/xacro">
     <!-- 属性封装 -->
     <xacro:arg name="gpu" default="true"/>
+    <!-- <xacro:arg name="organize_cloud" default="true"/> -->
     <xacro:property name="gpu" value="$(arg gpu)" />
-    <xacro:arg name="organize_cloud" default="true"/>
-    <xacro:property name="organize_cloud" value="$(arg organize_cloud)" />
+    <!-- <xacro:property name="organize_cloud" value="$(arg organize_cloud)" /> -->
+    <!-- 加载转动惯量描述 -->
     <xacro:include filename="$(find robot_description)/urdf/my_head.xacro" />
+    <!-- 加载底盘描述 -->
     <xacro:include filename="$(find robot_description)/urdf/my_base.xacro" />
-    <xacro:include filename="$(find robot_description)/urdf/my_camera.xacro" />
     <xacro:include filename="$(find robot_description)/urdf/move.xacro" />
     <!-- 更新结构信息，以laser_support + velodyne 为构建，不需要自己写雷达仿真的xacro文件 -->
@@ -16,9 +17,11 @@
     <xacro:include filename="$(find robot_description)/urdf/laser_support.xacro" />
     <xacro:include filename="$(find velodyne_description)/urdf/VLP-16.urdf.xacro"/>
-    <xacro:VLP-16 parent="support" name="velodyne" topic="/velodyne_points" organize_cloud="${organize_cloud}" hz="10" samples="440" gpu="${gpu}">
+    <xacro:VLP-16 parent="support" name="velodyne" topic="/velodyne_points" hz="10" samples="440" gpu="${gpu}">
           <origin xyz="0 0 ${support_length/2}" rpy="0 0 0" />
     </xacro:VLP-16>
     <!-- IMU 模块 -->
     <xacro:include filename="$(find robot_description)/urdf/my_imu.xacro"/>
+    <!-- 实例化 -->
+    <xacro:imu prefix="imu"/>
     <!-- 摄像头模块 -->
     <xacro:include filename="$(find robot_description)/urdf/my_camera.xacro" />
