Commit message: 尝试创建厂区地图

File: src/robot_description/urdf/my_base.xacro (robot description, xacro)
@@ -10,5 +10,5 @@
     <!-- 封装变量、常量 -->
     <!-- PI 值设置精度需要高一些，否则后续车轮翻转量计算时，可能会出现肉眼不能察觉的车轮倾斜，从而导致模型抖动 -->
-    <xacro:property name="PI" value="3.1415926"/>
+    <xacro:property name="PI" value="3.1415926535897932384626" />
     <!-- 宏:黑色设置 -->
     <material name="black">
@@ -17,8 +17,8 @@
     <!-- 底盘属性 -->
     <xacro:property name="base_footprint_radius" value="0.001" /> <!-- base_footprint 半径  -->
-    <xacro:property name="base_link_radius" value="0.1" /> <!-- base_link 半径 -->
-    <xacro:property name="base_link_length" value="0.08" /> <!-- base_link 长 -->
+    <xacro:property name="base_link_radius" value="0.5" /> <!-- base_link 半径 -->
+    <xacro:property name="base_link_length" value="0.2" /> <!-- base_link 长 -->
     <xacro:property name="earth_space" value="0.015" /> <!-- 离地间距 -->
-    <xacro:property name="base_link_m" value="0.5" /> <!-- 质量  -->
+    <xacro:property name="base_link_m" value="10" /> <!-- 质量  -->
     <!-- 底盘 -->
     <link name="base_footprint">
@@ -59,5 +59,5 @@
     <xacro:property name="wheel_radius" value="0.0325" /><!-- 半径 -->
     <xacro:property name="wheel_length" value="0.015" /><!-- 宽度 -->
-    <xacro:property name="wheel_m" value="0.05" /> <!-- 质量  -->
+    <xacro:property name="wheel_m" value="0.5" /> <!-- 质量  -->
     <!-- 驱动轮宏实现 -->
     <xacro:macro name="add_wheels" params="name flag">
@@ -93,5 +93,5 @@
     <!-- 支撑轮属性 -->
     <xacro:property name="support_wheel_radius" value="0.0075" /> <!-- 支撑轮半径 -->
-    <xacro:property name="support_wheel_m" value="0.03" /> <!-- 质量  -->
+    <xacro:property name="support_wheel_m" value="0.5" /> <!-- 质量  -->
     <!-- 支撑轮宏 -->
     <xacro:macro name="add_support_wheel" params="name flag" >

File: src/robot_description/urdf/my_laser.xacro (robot description, xacro)
@@ -4,5 +4,5 @@
 <robot name="my_laser" xmlns:xacro="http://wiki.ros.org/xacro">
     <!-- 雷达支架 -->
-    <xacro:property name="support_length" value="0.15" /> <!-- 支架长度 -->
+    <xacro:property name="support_length" value="0.10" /> <!-- 支架长度 -->
     <xacro:property name="support_radius" value="0.01" /> <!-- 支架半径 -->
     <xacro:property name="support_x" value="0.0" /> <!-- 支架安装的x坐标 -->
